File: Radio HAT/Radio HAT.kicad_sch (KiCad schematic)
At the start: 27 parts, among them J1 Raspberry_Pi_2_3, J2 Coax SMA, J3 Barrel_Jack, J4 VCC, J5 6V, J6 GND, J7 V_RF, U1 RFM98PW, U2 AZ2185D-ADJTRG1

Commit message: Changes for v1.2
Parts:
- added H3, H4: M, MountingHole:MountingHole_2.7mm_M2.5_Pad_Via, symbol Mechanical:MountingHole_Pad
- added R10, R11, R12, R13, R14, R9: 0, Resistor_SMD:R_0805_2012Metric_Pad1.20x1.40mm_HandSolder, symbol Device:R
- added R15: DNP, Resistor_SMD:R_0805_2012Metric_Pad1.20x1.40mm_HandSolder, symbol Device:R
Connections:
- net +3V3: now also R15.1; no longer C5.1, C6.1, U1.9 (3.3V)
- net GND: now also H3.1, H4.1
- net RF_DIO0: now also R9.2; no longer U1.6 (GPIO_0)
- net RF_DIO1: now also R10.2; no longer U1.7 (GPIO_1)
- net RF_DIO2: now also R11.2; no longer U1.8 (GPIO_2)
- net RF_DIO3: now also R12.2; no longer U1.3 (GPIO_3)
- net RF_DIO4: now also R13.2; no longer U1.4 (GPIO_4)
- net RF_DIO5: now also R14.2; no longer U1.15 (GPIO_5)
- new net: R12.1, U1.3 (GPIO_3)
- new net: R10.1, U1.7 (GPIO_1)
- new net: R13.1, U1.4 (GPIO_4)
- new net: R14.1, U1.15 (GPIO_5)
- new net: R9.1, U1.6 (GPIO_0)
- new net: R11.1, U1.8 (GPIO_2)
- new net RF_3V3: C5.1, C6.1, R15.2, U1.9 (3.3V)
Other:
- note added: "R9-R14 are 0-ohm resistors for connecting/disconnecting GPIO"
- moved on the sheet: C5, C6, D1, H1, H2, J1, J2, J4, J5, J6, J7, R1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

Commit message: Changes for v1.2
Parts:
- added J8: GPIO, TerminalBlock_TE-Connectivity:TerminalBlock_TE_282834-4_1x04_P2.54mm_Horizontal, symbol Connector_Generic:Conn_01x04
- added Q1: NMOS, Package_TO_SOT_SMD:SOT-23-3, symbol Simulation_SPICE:NMOS
Connections:
- net +6V: now also Q1.1 (D)
- net GND: now also J8.2 (Pin_2), J8.4 (Pin_4)
- net RX_EN: now reaches J1.15 (GPIO22)
- net RX_EN: now also J8.3 (Pin_3)
- net TX_EN: now reaches J1.16 (GPIO23)
- net TX_EN: now also Q1.2 (G)
- new net: J8.1 (Pin_1), Q1.3 (S)
- no-connect marks 20 -> 18
Changed lines of the file:
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@@
   (junction (at 176.53 142.24) (diameter 0) (color 0 0 0 0)
+  )
+  (junction (at 223.52 53.34) (diameter 0) (color 0 0 0 0)
   )
   (junction (at 189.23 67.31) (diameter 0) (color 0 0 0 0)
@@
   (no_connect (at 204.47 82.55))
   (no_connect (at 163.83 115.57))
-  (no_connect (at 163.83 113.03))
-  (no_connect (at 163.83 110.49))
-  (no_connect (at 163.83 92.71))
   (no_connect (at 179.07 72.39))
   (no_connect (at 163.83 118.11))
@@
   (no_connect (at 163.83 82.55))
   (no_connect (at 163.83 95.25))
+  (no_connect (at 163.83 92.71))
   (no_connect (at 204.47 97.79))
   (no_connect (at 181.61 72.39))
@@
     (stroke (width 0) (type default))
   )
+  (wire (pts (xy 153.67 113.03) (xy 163.83 113.03))
+    (stroke (width 0) (type default))
+  )
   (wire (pts (xy 55.88 104.14) (xy 55.88 105.41))
     (stroke (width 0) (type default))
@@
     (stroke (width 0) (type default))
   )
+  (wire (pts (xy 231.14 48.26) (xy 223.52 48.26))
+    (stroke (width 0) (type default))
+  )
   (wire (pts (xy 74.93 52.07) (xy 74.93 53.34))
     (stroke (width 0) (type default))
@@
     (stroke (width 0) (type default))
   )
+  (wire (pts (xy 229.87 45.72) (xy 231.14 45.72))
+    (stroke (width 0) (type default))
+  )
   (wire (pts (xy 186.69 138.43) (xy 186.69 142.24))
     (stroke (width 0) (type default))
@@
     (stroke (width 0) (type default))
   )
+  (wire (pts (xy 223.52 53.34) (xy 223.52 57.15))
+    (stroke (width 0) (type default))
+  )
   (wire (pts (xy 204.47 110.49) (xy 214.63 110.49))
     (stroke (width 0) (type default))
@@
     (stroke (width 0) (type default))
   )
+  (wire (pts (xy 223.52 53.34) (xy 231.14 53.34))
+    (stroke (width 0) (type default))
+  )
   (wire (pts (xy 176.53 142.24) (xy 179.07 142.24))
     (stroke (width 0) (type default))
@@
     (stroke (width 0) (type default))
   )
+  (wire (pts (xy 229.87 44.45) (xy 229.87 45.72))
+    (stroke (width 0) (type default))
+  )
   (wire (pts (xy 204.47 118.11) (xy 214.63 118.11))
     (stroke (width 0) (type default))
@@
     (stroke (width 0) (type default))
   )
+  (wire (pts (xy 215.9 39.37) (xy 222.25 39.37))
+    (stroke (width 0) (type default))
+  )
   (wire (pts (xy 71.12 104.14) (xy 71.12 105.41))
     (stroke (width 0) (type default))
   )
+  (wire (pts (xy 223.52 48.26) (xy 223.52 53.34))
+    (stroke (width 0) (type default))
+  )
+  (wire (pts (xy 229.87 33.02) (xy 229.87 34.29))
+    (stroke (width 0) (type default))
+  )
   (wire (pts (xy 179.07 138.43) (xy 179.07 142.24))
     (stroke (width 0) (type default))
@@
     (stroke (width 0) (type default))
   )
+  (wire (pts (xy 153.67 110.49) (xy 163.83 110.49))
+    (stroke (width 0) (type default))
+  )
   (wire (pts (xy 173.99 142.24) (xy 176.53 142.24))
     (stroke (width 0) (type default))
@@
   )
   (wire (pts (xy 114.3 121.92) (xy 115.57 121.92))
+    (stroke (width 0) (type default))
+  )
+  (wire (pts (xy 224.79 50.8) (xy 231.14 50.8))
     (stroke (width 0) (type default))
   )
@@
     (effects (font (size 1.27 1.27)) (justify left bottom))
   )
+  (label "TX_EN" (at 215.9 39.37 0) (fields_autoplaced)
+    (effects (font (size 1.27 1.27)) (justify left bottom))
+  )
   (label "V_RF" (at 95.25 87.63 0) (fields_autoplaced)
+    (effects (font (size 1.27 1.27)) (justify left bottom))
+  )
+  (label "RX_EN" (at 153.67 110.49 0) (fields_autoplaced)
     (effects (font (size 1.27 1.27)) (justify left bottom))
   )
@@
     (effects (font (size 1.27 1.27)) (justify left bottom))
   )
+  (label "RX_EN" (at 224.79 50.8 0) (fields_autoplaced)
+    (effects (font (size 1.27 1.27)) (justify left bottom))
+  )
+  (label "TX_EN" (at 153.67 113.03 0) (fields_autoplaced)
+    (effects (font (size 1.27 1.27)) (justify left bottom))
+  )
   (label "RF_3V3" (at 73.66 114.3 0) (fields_autoplaced)
     (effects (font (size 1.27 1.27)) (justify left bottom))
@@
     )
   )
+  (symbol (lib_id "power:+6V") (at 229.87 33.02 0) (unit 1)
+    (in_bom yes) (on_board yes) (dnp no) (fields_autoplaced)
+    (property "Reference" "#PWR025" (at 229.87 36.83 0)
+      (effects (font (size 1.27 1.27)) hide)
+    )
+    (property "Value" "+6V" (at 229.87 29.21 0)
+      (effects (font (size 1.27 1.27)))
+    )
+    (property "Footprint" "" (at 229.87 33.02 0)
+      (effects (font (size 1.27 1.27)) hide)
+    )
+    (property "Datasheet" "" (at 229.87 33.02 0)
+      (effects (font (size 1.27 1.27)) hide)
+    )
+    (pin "1")
+    (instances
+      (project "Radio HAT"
+        (path "/e833ba5c-90ae-4111-9eec-1a872963763a"
+          (reference "#PWR025") (unit 1)
+        )
+      )
+    )
+  )
   (symbol (lib_id "power:GND") (at 104.14 67.31 0) (unit 1)
     (in_bom yes) (on_board yes) (dnp no)
@@
     )
   )
+  (symbol (lib_id "power:GND") (at 223.52 57.15 0) (unit 1)
+    (in_bom yes) (on_board yes) (dnp no)
+    (property "Reference" "#PWR026" (at 223.52 63.5 0)
+      (effects (font (size 1.27 1.27)) hide)
+    )
+    (property "Value" "GND" (at 223.52 62.23 0)
+      (effects (font (size 1.27 1.27)))
+    )
+    (property "Footprint" "" (at 223.52 57.15 0)
+      (effects (font (size 1.27 1.27)) hide)
+    )
+    (property "Datasheet" "" (at 223.52 57.15 0)
+      (effects (font (size 1.27 1.27)) hide)
+    )
+    (pin "1")
+    (instances
+      (project "Radio HAT"
+        (path "/e833ba5c-90ae-4111-9eec-1a872963763a"
+          (reference "#PWR026") (unit 1)
+        )
+      )
+    )
+  )
   (symbol (lib_id "power:GND") (at 140.97 134.62 0) (unit 1)
     (in_bom yes) (on_board yes) (dnp no)
@@
         (path "/e833ba5c-90ae-4111-9eec-1a872963763a"
           (reference "C6") (unit 1)
+        )
+      )
+    )
+  )
+  (symbol (lib_id "Connector_Generic:Conn_01x04") (at 236.22 48.26 0) (unit 1)
+    (in_bom yes) (on_board yes) (dnp no) (fields_autoplaced)
+    (property "Reference" "J8" (at 238.76 48.895 0)
+      (effects (font (size 1.27 1.27)) (justify left))
+    )
+    (property "Value" "GPIO" (at 238.76 51.435 0)
+      (effects (font (size 1.27 1.27)) (justify left))
+    )
+    (property "Footprint" "TerminalBlock_TE-Connectivity:TerminalBlock_TE_282834-4_1x04_P2.54mm_Horizontal" (at 236.22 48.26 0)
+      (effects (font (size 1.27 1.27)) hide)
+    )
+    (property "Datasheet" "~" (at 236.22 48.26 0)
+      (effects (font (size 1.27 1.27)) hide)
+    )
+    (pin "1")
+    (pin "2")
+    (pin "3")
+    (pin "4")
+    (instances
+      (project "Radio HAT"
+        (path "/e833ba5c-90ae-4111-9eec-1a872963763a"
+          (reference "J8") (unit 1)
         )
       )
@@
         )
       )
+    )
+  )
+  (symbol (lib_id "Simulation_SPICE:NMOS") (at 227.33 39.37 0) (unit 1)
+    (in_bom yes) (on_board yes) (dnp no) (fields_autoplaced)
+    (property "Reference" "Q1" (at 233.68 38.735 0)
+      (effects (font (size 1.27 1.27)) (justify left))
+    )
+    (property "Value" "NMOS" (at 233.68 41.275 0)
+      (effects (font (size 1.27 1.27)) (justify left))
+    )
+    (property "Footprint" "Package_TO_SOT_SMD:SOT-23-3" (at 232.41 36.83 0)
+      (effects (font (size 1.27 1.27)) hide)
+    )
+    (property "Datasheet" "https://ngspice.sourceforge.io/docs/ngspice-manual.pdf" (at 227.33 52.07 0)
+      (effects (font (size 1.27 1.27)) hide)
+    )
+    (property "Sim.Device" "NMOS" (at 227.33 56.515 0)
+      (effects (font (size 1.27 1.27)) hide)
+    )
+    (property "Sim.Type" "VDMOS" (at 227.33 58.42 0)
+      (effects (font (size 1.27 1.27)) hide)
+    )
+    (property "Sim.Pins" "1=D 2=G 3=S" (at 227.33 54.61 0)
+      (effects (font (size 1.27 1.27)) hide)
+    )
+    (pin "1")
+    (pin "2")
+    (pin "3")
+    (instances
+      (project "Radio HAT"
+        (path "/e833ba5c-90ae-4111-9eec-1a872963763a"
+          (reference "Q1") (unit 1)
+        )
+      )

Commit message: Fixed TX and RX enable circuits
Parts:
- added R16, R17: DNP, Resistor_SMD:R_0805_2012Metric_Pad1.20x1.40mm_HandSolder, symbol Device:R
Connections:
- net +6V: no longer Q1.1 (D)
- net GND: now also Q1.3 (S)
- net RX_EN: now also R16.2; no longer J1.15 (GPIO22)
- net TX_EN: now also J8.1 (Pin_1), R17.2; no longer J1.16 (GPIO23), Q1.2 (G)
- new net: Q1.1 (D), R17.1
- new net PI_RX_CTRL: J1.15 (GPIO22), R16.1
- new net PI_TX_CTRL: J1.16 (GPIO23), Q1.2 (G)
Other:
- note added: "Populate R16 to enable GPIO control for RX enable Populate R17 to enable GPIO control for TX enable"
- moved on the sheet: J8, Q1
